File: layout-diag/layout-diag.kicad_pcb (KiCad board)
At the start: 2 copper layers, 0 parts

Commit message: PCB Updates and added panel-fw project.
Other:
- board text added: "FEED[A+]"
- board text added: "FEED[A-]"
- board text added: "FEED[B+]"
- board text added: "FEED[B-]"
- board text added: "FEED[C+]"
- board text added: "FEED[C-]"
- board text added: "FEED[D+]"
- board text added: "FEED[D-]"
- board text added: "FEED[E+]"
- board text added: "FEED[F+]"
- board text added: "FEED[G+]"
- board text added: "FEED[H+]"
- board text added: "FEED[I-]"
- board text added: "FEED[J-]"
- board text removed: "FEED#A"
- board text removed: "FEED#B"
- board text removed: "FEED#C"
- board text removed: "FEED#D"
- board text removed: "FEED#E"
- board text removed: "FEED#F"
- board text removed: "FEED#G"
- board text removed: "FEED#H"
- board text removed: "FEED#I"
- board text removed: "FEED#J"
- board text removed: "FEED#K"
- board text removed: "FEED#L"
- board text removed: "FEED#M"
- board text removed: "FEED#N"
- board text removed: "FEED#O"
- board text removed: "FEED#P"
- board text removed: "FEED#Q"
- board text removed: "FEED#R"
- board text removed: "FEED#S"
- board text removed: "FEED#T"
- board text removed: "FEED#U"
- board text removed: "FEED#V"
- board text removed: "FEED#X"
